File: hardwarez/Linx/Linx.kicad_sch (KiCad schematic)
At the start: 1 part, among them IC1 6502

Commit message: hardware_stuff
Parts:
- added R1: R, Resistor_THT:R_Axial_DIN0204_L3.6mm_D1.6mm_P5.08mm_Horizontal, symbol Device:R
- added SW1: SW_MEC_5G, Button_Switch_SMD:SW_MEC_5GSH9, symbol Switch:SW_MEC_5G
Connections:
- net GND: now reaches IC1.1
- net GND: now also IC1.21, SW1.3 (B), SW1.4 (B)
- net VCC: now reaches IC1.2 (RDY)
- net VCC: now also IC1.4 (IRQ), IC1.6 (NMI), IC1.8, R1.1
- net at IC1.40 (RESET): now also R1.2, SW1.1 (A), SW1.2 (A)
Other:
- moved on the sheet: IC1A, IC1B, IC1C, IC1D

Commit message: more hardware stuffs
Parts:
- added U1: 4028, symbol 4xxx:4028
Connections:
- net GND: now also U1.8 (VSS)
- net VCC: now also U1.16 (VDD)
Other:
- moved on the sheet: IC1A, IC1B, IC1C, IC1D, R1, SW1

Commit message: Linx
Parts:
- added U2: 27C256, Package_DIP:DIP-28_W15.24mm, symbol Memory_EPROM:27C256
- added Y1: Crystal, Crystal:Crystal_HC18-U_Vertical, symbol Device:Crystal
Connections:
- net GND: now also U2.14 (GND), U2.26 (A13), U2.27 (A14)
- net VCC: now also U2.28 (VCC), Y1.2
- net at U1.10 (A): now also IC1.23 (A13)
- net at U1.12 (C): now also IC1.25 (A15)
- net at U1.13 (B): now also IC1.24 (A14)
- net at U1.3 (S0): now also U2.20 (~{CE}), U2.22 (~{OE})
- net at IC1.10 (A1): now also U2.9 (A1)
- net at IC1.11 (A2): now also U2.8 (A2)
- net at IC1.12 (A3): now also U2.7 (A3)
- net at IC1.13 (A4): now also U2.6 (A4)
- net at IC1.14 (A5): now also U2.5 (A5)
- net at IC1.15 (A6): now also U2.4 (A6)
- net at IC1.16 (A7): now also U2.3 (A7)
- net at IC1.17 (A8): now also U2.25 (A8)
- net at IC1.18 (A9): now also U2.24 (A9)
- net at IC1.19 (A10): now also U2.21 (A10)
- net at IC1.20 (A11): now also U2.23 (A11)
- net at IC1.22 (A12): now also U2.2 (A12)
- net at IC1.26 (DB7): now also U2.19 (D7)
- net at IC1.27 (DB6): now also U2.18 (D6)
- net at IC1.28 (DB5): now also U2.17 (D5)
- net at IC1.29 (DB4): now also U2.16 (D4)
- net at IC1.30 (DB3): now also U2.15 (D3)
- net at IC1.31 (DB2): now also U2.13 (D2)
- net at IC1.32 (DB1): now also U2.12 (D1)
- net at IC1.33 (DB0): now also U2.11 (D0)
- net at IC1.37 (PH0): now also Y1.1
- net at IC1.9 (A0): now also U2.10 (A0)
